File: Duskpad.kicad_pcb (KiCad board)
At the start: 2 copper layers, 3.6 x 3.2 mm, 50 parts, among them J1 OLED display, SW1 SW_Push, SW10 SW_Push, SW11 SW_Push, SW12 SW_Push, SW13 SW_Push, SW14 SW_Push, SW15 SW_Push, SW16 SW_Push, SW2 SW_Push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

Commit message: did the pcb design
Parts:
- added D33: SK6812MINI-E, LED_SMD:LED_SK6812MINI-E_3.2x2.8mm_P1.5mm_ReverseMount, F.Cu at (99.3, 30.1)
- added D34: SK6812MINI-E, LED_SMD:LED_SK6812MINI-E_3.2x2.8mm_P1.5mm_ReverseMount, F.Cu at (99.3, 34.9)
- added D35: SK6812MINI-E, LED_SMD:LED_SK6812MINI-E_3.2x2.8mm_P1.5mm_ReverseMount, F.Cu at (99.3, 39.8)
- added D36: SK6812MINI-E, LED_SMD:LED_SK6812MINI-E_3.2x2.8mm_P1.5mm_ReverseMount, F.Cu at (99.3, 44.7)
- D1, D10, D11, D12, D13, D14, D15, D16, D2, D3, D4, D5, D6, D7, D8, D9: moved to B.Cu
- J1: footprint Connector_PinHeader_2.54mm:PinHeader_1x04_P2.54mm_Vertical -> footprints:SSD1306-0.91-OLED-4pin-128x32
- moved J1 140.9 mm to (109.2, 32.2)
- moved U1 127.1 mm to (80.5, 36.8)
- moved SW13 118.5 mm to (83.2, 109.2)
- moved D13 103.3 mm to (90.1, 117.9), turned to 90 degrees
- moved D9 101.9 mm to (90.1, 99.4), turned to 90 degrees
- moved D5 100.6 mm to (90.1, 80.4), turned to 90 degrees
- moved D1 99.6 mm to (90.1, 61.4), turned to 90 degrees
- moved SW14 91.7 mm to (102.2, 109.2)
- moved SW9 91.7 mm to (83.2, 90.2)
- moved D14 84.2 mm to (109.1, 117.9), turned to 90 degrees
- moved D10 82.7 mm to (109.1, 99.4), turned to 90 degrees
- moved D6 80.9 mm to (109.6, 80.4), turned to 90 degrees
- moved D2 79.8 mm to (109.6, 61.4), turned to 90 degrees
- moved D15 65.3 mm to (128.1, 117.9), turned to 90 degrees
- moved SW10 65.0 mm to (102.2, 90.2)
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Connections:
- net Net-(D17-DIN) renamed DIN
- D29 pad 2: unconnected-(D29-DIN-Pad2) -> Net-(D29-DIN)
Routing:
- net GND: track 0.00 -> 469.5 mm, vias 0 -> 46
- net VCC(5V): track 0.00 -> 425.5 mm, vias 0 -> 20
- net Row 4: track 0.00 -> 151.2 mm, vias 0 -> 2
- net Row 3: track 0.00 -> 134.9 mm, vias 0 -> 2
- net Net-(D29-DIN): track 0.00 -> 124.5 mm
- net Row 2: track 0.00 -> 114.7 mm, vias 0 -> 2
- net Colunm 4: track 0.00 -> 112.7 mm, vias 0 -> 4
- net Net-(J1-Pin_3): track 0.00 -> 98.9 mm
- net Net-(J1-Pin_4): track 0.00 -> 96.4 mm
- net Colunm 3: track 0.00 -> 95.8 mm, vias 0 -> 2
- net Row 1: track 0.00 -> 93.8 mm, vias 0 -> 2
- net VCC(3V): track 0.00 -> 78.3 mm, vias 0 -> 2
- net Colunm 2: track 0.00 -> 77.1 mm
- net Colunm 1: track 0.00 -> 74.9 mm
- net Net-(D21-DIN): track 0.00 -> 22.4 mm
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Other:
- board size 3.6 x 3.2 mm -> 82.5 x 100 mm
